Commit message: commiting urdf changes

File: src/mushr_description/urdf/racecar.urdf (robot description, URDF)
Before this commit: robot mushr_tx2, 13 links, 12 joints
Links:
- added link laser, mass 0.130; collision box size=0.010 0.010 0.010; visual box size=0.05 0.05 0.07
Joints:
- added joint laser_joint: type fixed, parent base_link, child laser, origin xyz=0.03975 0.0 0.180 rpy=0 0 0
